Commit message: update

File: src/articubot_one/description/robot.urdf.xacro (robot description, xacro)
@@ -5,3 +5,15 @@
     <xacro:include filename = "gazebo_control.xacro" />
     <xacro:include filename = "lidar.xacro" />
+    <xacro:include filename = "gripper.xacro" />
+    <xacro:include filename="gripper_tranmission.xacro" />
+    <xacro:include filename="gazebo_plugin.xacro"/>
+    <xacro:robot_controller/>
+    <ros2_control name="gripper_robot_gazebo_system" type="system">
+        <hardware>
+            <plugin>gazebo_ros2_control/GazeboSystem</plugin>
+        </hardware>
+        <xacro:gripper_vertical_tranmission/>
+        <xacro:gripper_finger_left_tranmission/>
+        <xacro:gripper_finger_right_tranmission/>
+    </ros2_control>
 </robot>

File: src/articubot_one/description/robot_core.xacro (robot description, xacro)
@@ -5,19 +5,18 @@
      <color rgba="1 1 1 1" />
  </material>
- <material name="orange">
-     <color rgba="1 0.3 0.1 1"/>
- </material>
- <material name="blue">
-     <color rgba="0.2 0.2 1 1"/>
- </material>
  <material name="black">
      <color rgba="0 0 0 1"/>
- </material>
- <material name="red">
-     <color rgba="1 0 0 1"/>
  </material>
  <!-- BASE LINK -->
  <link name="base_link">
  </link>
+ <!-- BASE_FOOTPRINT LINK -->
+<joint name="base_footprint_joint" type="fixed">
+ <parent link="base_link"/>
+ <child link="base_footprint"/>
+ <origin xyz="0 0 0" rpy="0 0 0"/>
+</joint>
+<link name="base_footprint">
+</link>
  <joint name="chassis_joint" type="fixed">
  <parent link="base_link"/>
@@ -39,5 +38,5 @@
     </geometry>
 </collision>
-<xacro:inertial_box mass="30.0" x="0.451" y="0.451" z="0.2">
+<xacro:inertial_box mass="200" x="0.451" y="0.451" z="0.2">
       <origin xyz="0.125 0 0.0" rpy="0 0 0"/>
   </xacro:inertial_box>
@@ -58,5 +57,5 @@
         <cylinder length="0.04" radius="0.1" />
     </geometry>
-    <material name="blue"/>
+    <material name="black"/>
 </visual>
 <collision>
@@ -70,5 +69,5 @@
 </link>
 <gazebo reference="left_wheel01">
-   <material>Gazebo/Blue</material>
+   <material>Gazebo/Black</material>
 </gazebo>
 <!-- LEFT WHEEL02 -->
@@ -84,5 +83,5 @@
         <cylinder length="0.04" radius="0.1" />
     </geometry>
-    <material name="orange"/>
+    <material name="black"/>
 </visual>
 <collision>
@@ -96,5 +95,5 @@
 </link>
 <gazebo reference="left_wheel02">
-   <material>Gazebo/Orange</material>
+   <material>Gazebo/Black</material>
 </gazebo>
 <!-- RIGHT WHEEL01 -->
@@ -136,5 +135,5 @@
         <cylinder length="0.04" radius="0.1" />
     </geometry>
-    <material name="red"/>
+    <material name="black"/>
 </visual>
 <collision>
@@ -148,5 +147,5 @@
 </link>
 <gazebo reference="right_wheel02">
-   <material>Gazebo/Red</material>
+   <material>Gazebo/Black</material>
 </gazebo>
 <!-- CASTER WHEEL
