Commit message: finish01

File: src/articubot_one/description/gripper.xacro (robot description, xacro)
@@ -55,6 +55,6 @@
                 <friction>
                     <ode>
-                        <mu>2.0</mu>  <!-- Increase primary friction -->
-                        <mu2>2.0</mu2>  <!-- Increase secondary friction -->
+                        <mu>50</mu>  <!-- Increase primary friction -->
+                        <mu2>50</mu2>  <!-- Increase secondary friction -->
                     </ode>
                 </friction>
@@ -92,6 +92,6 @@
                 <friction>
                     <ode>
-                        <mu>2.0</mu>  <!-- Increase primary friction -->
-                        <mu2>2.0</mu2>  <!-- Increase secondary friction -->
+                        <mu>50</mu>  <!-- Increase primary friction -->
+                        <mu2>50</mu2>  <!-- Increase secondary friction -->
                     </ode>
                 </friction>
@@ -128,5 +128,5 @@
         <axis xyz="1 0 0"/>
         <limit effort="100" lower="0" upper="0.1" velocity="0.1"/>
-        <dynamics damping="20.0" friction="2.0"/>
+        <dynamics damping="20.0" friction="1.0"/>
     </joint>
     <joint name="gripper_finger_right_joint" type="prismatic">
@@ -136,5 +136,5 @@
         <axis xyz="1 0 0"/>
         <limit effort="100" lower="-0.1" upper="0" velocity="0.1"/>
-        <dynamics damping="20.0" friction="2.0"/>
+        <dynamics damping="20.0" friction="1.0"/>
     </joint>
     <!-- Gazebo Simulation for Gripper -->

File: src/articubot_one/description/lidar.xacro (robot description, xacro)
@@ -26,5 +26,5 @@
         <sensor name="laser" type="ray">
             <pose> 0 0 0 0 0 0 </pose>
-            <visualize>true</visualize>
+            <visualize>false</visualize>
             <update_rate>10</update_rate>
             <ray>
